File: _autosave-solder-2nd-attempt.kicad_sch (KiCad schematic)
At the start: 18 parts, among them Q1 NPN, Q2 NPN, Q3 NPN, SW1 SW_Push

Commit message: updated schematic + pcb
Parts:
- C1: value C -> 10uF
- C2: value C -> 470nF
- R1, R2: value R -> 470
- R4: value R -> 220
- R5: value R -> 4.7K
- R6: value R -> 100K
- R7: value R -> 47K
- R8: value R -> 2.2M
Connections:
- net at C1.1, Q1.2 (B), R3.1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: now also Q1.1 (C)
Changed lines of the file:
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@@
+	)
+	(junction
+		(at 162.56 67.31)
+		(diameter 0)
+		(color 0 0 0 0)
 	)
 	(junction
@@
 	(wire
 		(pts
-			(xy 176.53 66.04) (xy 176.53 74.93)
-		)
-		(stroke
-			(width 0)
-			(type default)
-		)
-	)
-	(wire
-		(pts
 			(xy 162.56 80.01) (xy 168.91 80.01)
 		)
@@
 	(wire
 		(pts
+			(xy 176.53 67.31) (xy 176.53 74.93)
+		)
+		(stroke
+			(width 0)
+			(type default)
+		)
+	)
+	(wire
+		(pts
 			(xy 90.17 106.68) (xy 99.06 106.68)
 		)
@@
 	(wire
 		(pts
-			(xy 162.56 66.04) (xy 176.53 66.04)
+			(xy 162.56 67.31) (xy 176.53 67.31)
 		)
 		(stroke
@@
 			)
 		)
-		(property "Value" "R"
+		(property "Value" "2.2M"
 			(at 68.58 125.7299 0)
 			(effects
@@
 			)
 		)
-		(property "Value" "C"
+		(property "Value" "470nF"
 			(at 50.8 123.1899 0)
 			(effects
@@
 			)
 		)
-		(property "Value" "R"
+		(property "Value" "4.7K"
 			(at 92.71 64.7699 0)
 			(effects
@@
 			)
 		)
-		(property "Value" "R"
+		(property "Value" "47K"
 			(at 49.53 102.8699 0)
 			(effects
@@
 			)
 		)
-		(property "Value" "R"
+		(property "Value" "220"
 			(at 109.22 62.2299 0)
 			(effects
@@
 			)
 		)
-		(property "Value" "R"
+		(property "Value" "470"
 			(at 219.71 83.8199 0)
 			(effects
@@
 			)
 		)
-		(property "Value" "R"
+		(property "Value" "470"
 			(at 196.342 78.74 0)
 			(effects
@@
 			)
 		)
-		(property "Value" "R"
+		(property "Value" "100K"
 			(at 101.6 90.17 90)
 			(effects
@@
 			)
 		)
-		(property "Value" "C"
+		(property "Value" "10uF"
 			(at 180.34 104.1399 0)
 			(effects
